Commit message: Add mission framework, field map, navigation, and gantry safety improvements
- robot_missions: full PlantingMission lifecycle (validate/plan/execute/report),
  ExecutionEngine with Z-retract-before-XY, FlatGroundDepthSensor, GripperTool,
  MissionManager navigation-to-start, action server with 2 Hz feedback, abort guard
- robot_field: new package — single source of truth for field layout (field_config.yaml,
  mission_zones.yaml); HTTP API at /api/field_config and /api/mission_zones
- robot_navigation: NavigationProvider interface + OdometryNavigator (0.1 m/s, odom feedback)
- robot_web_app: missions UI (canvas field map, 2-click zone placement, overlap validation,
  seed stats, ▶ Start / ■ Cancel per zone, rosbridge action goals + feedback)
- mks_servo_hardware: velocity caps in both modes, sqrt decel, soft position limits,
  homing false-success fix (any_motion tracking per motor), stale-offset guard
- robot_bringup: launch XML updated; JTC spawned after homing via --controller-manager-timeout 120
- MAP_ARCHITECTURE.md: field coordinate system, canvas rendering strategy, roadmap Steps 5-7

Co-Authored-By: Claude Sonnet 4.6 <noreply@anthropic.com>

File: src/robot_description/urdf/mobile_base.xacro (robot description, xacro)
@@ -16,4 +16,5 @@
     <xacro:property name="z_axis_travel" value="0.25" />
     <xacro:property name="wheel_radius" value="0.0825" />
+    <xacro:property name="wheel_width"  value="0.10"   />   <!-- tread width in Y (axle direction) -->
     ``----- LINKS -----
     <link name="base_footprint" />
